Commit message: feat: add camera and lidar links to rover

File: src/space_rover/urdf/rover.urdf.xacro (robot description, xacro)
@@ -9,4 +9,30 @@
     </visual>
   </link>
+    <!-- Camera -->
+  <link name="camera_link">
+    <visual>
+      <geometry>
+        <box size="0.05 0.05 0.05"/>
+      </geometry>
+    </visual>
+  </link>
+  <joint name="camera_joint" type="fixed">
+    <parent link="base_link"/>
+    <child link="camera_link"/>
+    <origin xyz="0.2 0 0.15"/>
+  </joint>
+  <!-- LIDAR -->
+  <link name="lidar_link">
+    <visual>
+      <geometry>
+        <cylinder radius="0.04" length="0.03"/>
+      </geometry>
+    </visual>
+  </link>
+  <joint name="lidar_joint" type="fixed">
+    <parent link="base_link"/>
+    <child link="lidar_link"/>
+    <origin xyz="0 0 0.2"/>
+  </joint>
   <!-- Wheels -->
   <!-- Left side -->

Commit message: feat: add space rover model

File: src/space_rover/urdf/rover.urdf.xacro (robot description, xacro)
@@ -1,85 +1,174 @@
 <?xml version="1.0"?>
 <robot name="rover" xmlns:xacro="http://www.ros.org/wiki/xacro">
-  <!-- Base -->
+  <!-- BASE -->
   <link name="base_link">
     <visual>
       <geometry>
-        <box size="0.6 0.4 0.15"/>
+        <box size="0.7 0.5 0.12"/>
       </geometry>
+	<material name="light_gray">
+  <color rgba="0.7 0.7 0.75 1"/>
+</material>
     </visual>
+<material name="accent">
+  <color rgba="0.9 0.6 0.1 1"/>
+</material>
+    <collision>
+      <geometry>
+        <box size="0.7 0.5 0.12"/>
+      </geometry>
+    </collision>
+    <inertial>
+      <mass value="10.0"/>
+      <inertia ixx="1" iyy="1" izz="1" ixy="0" ixz="0" iyz="0"/>
+    </inertial>
   </link>
-    <!-- Camera -->
-  <link name="camera_link">
-    <visual>
-      <geometry>
-        <box size="0.05 0.05 0.05"/>
-      </geometry>
-    </visual>
-  </link>
-  <joint name="camera_joint" type="fixed">
-    <parent link="base_link"/>
-    <child link="camera_link"/>
-    <origin xyz="0.2 0 0.15"/>
-  </joint>
+  <link name="mast_link">
+  <visual>
+    <geometry>
+      <cylinder radius="0.03" length="0.4"/>
+    </geometry>
+    <material name="white">
+      <color rgba="0.9 0.9 0.9 1"/>
+    </material>
+  </visual>
+</link>
+<joint name="mast_joint" type="fixed">
+  <parent link="base_link"/>
+  <child link="mast_link"/>
+  <origin xyz="0.2 0 0.3"/>
+</joint>
+  <!-- CAMERA -->
+<link name="camera_link">
+  <visual>
+    <geometry>
+      <box size="0.12 0.08 0.06"/>
+    </geometry>
+    <material name="blue">
+      <color rgba="0.1 0.3 1 1"/>
+    </material>
+  </visual>
+  <collision>
+    <geometry>
+      <box size="0.12 0.08 0.06"/>
+    </geometry>
+  </collision>
+  <inertial>
+    <mass value="0.5"/>
+    <inertia ixx="0.01" iyy="0.01" izz="0.01" ixy="0" ixz="0" iyz="0"/>
+  </inertial>
+</link>
+<link name="camera_lens">
+<visual>
+  <origin rpy="0 1.5707 0"/>
+  <geometry>
+    <cylinder radius="0.02" length="0.03"/>
+  </geometry>
+  <material name="black">
+    <color rgba="0 0 0 1"/>
+  </material>
+</visual>
+</link>
+<joint name="camera_lens_joint" type="fixed">
+  <parent link="camera_link"/>
+  <child link="camera_lens"/>
+  <origin xyz="0.06 0 0"/>
+</joint>
+<joint name="camera_joint" type="fixed">
+  <parent link="mast_link"/>
+  <child link="camera_link"/>
+  <origin xyz="0 0 0.18"/>
+</joint>
   <!-- LIDAR -->
   <link name="lidar_link">
     <visual>
       <geometry>
-        <cylinder radius="0.04" length="0.03"/>
+        <cylinder radius="0.05" length="0.05"/>
       </geometry>
+      <material name="black">
+        <color rgba="0.05 0.05 0.05 1"/>
+      </material>
     </visual>
+    <collision>
+      <geometry>
+        <cylinder radius="0.05" length="0.05"/>
+      </geometry>
+    </collision>
+    <inertial>
+      <mass value="0.5"/>
+      <inertia ixx="0.01" iyy="0.01" izz="0.01" ixy="0" ixz="0" iyz="0"/>
+    </inertial>
   </link>
   <joint name="lidar_joint" type="fixed">
     <parent link="base_link"/>
     <child link="lidar_link"/>
-    <origin xyz="0 0 0.2"/>
+    <origin xyz="0 0 0.18"/>
   </joint>
-  <!-- Wheels -->
-  <!-- Left side -->
-  <link name="front_left_wheel"><visual><geometry><cylinder radius="0.08" length="0.06"/></geometry></visual></link>
-  <link name="mid_left_wheel"><visual><geometry><cylinder radius="0.08" length="0.06"/></geometry></visual></link>
-  <link name="rear_left_wheel"><visual><geometry><cylinder radius="0.08" length="0.06"/></geometry></visual></link>
-  <!-- Right side -->
-  <link name="front_right_wheel"><visual><geometry><cylinder radius="0.08" length="0.06"/></geometry></visual></link>
-  <link name="mid_right_wheel"><visual><geometry><cylinder radius="0.08" length="0.06"/></geometry></visual></link>
-  <link name="rear_right_wheel"><visual><geometry><cylinder radius="0.08" length="0.06"/></geometry></visual></link>
-  <!-- Joints -->
-  <!-- Left wheels -->
-  <joint name="fl_joint" type="continuous">
+  <link name="left_arm">
+  <visual>
+    <geometry>
+      <box size="0.4 0.05 0.05"/>
+    </geometry>
+    <material name="gray"/>
+  </visual>
+</link>
+<joint name="left_arm_joint" type="fixed">
+  <parent link="base_link"/>
+  <child link="left_arm"/>
+  <origin xyz="0 0.25 -0.05"/>
+</joint>
+  <link name="solar_panel">
+  <visual>
+    <geometry>
+      <box size="0.5 0.3 0.02"/>
+    </geometry>
+    <material name="blue_dark">
+      <color rgba="0.1 0.1 0.4 1"/>
+    </material>
+  </visual>
+</link>
+<joint name="solar_joint" type="fixed">
+  <parent link="base_link"/>
+  <child link="solar_panel"/>
+  <origin xyz="-0.1 0 0.15"/>
+</joint>
+  <!-- WHEEL MACRO -->
+  <xacro:macro name="wheel" params="name x y">
+  <link name="${name}">
+    <visual>
+      <origin rpy="1.5707 0 0"/>
+      <geometry>
+        <cylinder radius="0.12" length="0.06"/>
+      </geometry>
+      <material name="wheel_black">
+        <color rgba="0.1 0.1 0.1 1"/>
+      </material>
+    </visual>
+    <collision>
+      <origin rpy="1.5707 0 0"/>
+      <geometry>
+        <cylinder radius="0.12" length="0.06"/>
+      </geometry>
+    </collision>
+    <inertial>
+      <mass value="1.0"/>
+      <inertia ixx="0.1" iyy="0.1" izz="0.1" ixy="0" ixz="0" iyz="0"/>
+    </inertial>
+  </link>
+  <joint name="${name}_joint" type="continuous">
     <parent link="base_link"/>
-    <child link="front_left_wheel"/>
-    <origin xyz="0.25 0.2 0"/>
+    <child link="${name}"/>
+    <origin xyz="${x} ${y} -0.12"/>
     <axis xyz="0 1 0"/>
   </joint>
-  <joint name="ml_joint" type="continuous">
-    <parent link="base_link"/>
-    <child link="mid_left_wheel"/>
-    <origin xyz="0 0.2 0"/>
-    <axis xyz="0 1 0"/>
-  </joint>
-  <joint name="rl_joint" type="continuous">
-    <parent link="base_link"/>
-    <child link="rear_left_wheel"/>
-    <origin xyz="-0.25 0.2 0"/>
-    <axis xyz="0 1 0"/>
-  </joint>
-  <!-- Right wheels -->
-  <joint name="fr_joint" type="continuous">
-    <parent link="base_link"/>
-    <child link="front_right_wheel"/>
-    <origin xyz="0.25 -0.2 0"/>
-    <axis xyz="0 1 0"/>
-  </joint>
-  <joint name="mr_joint" type="continuous">
-    <parent link="base_link"/>
-    <child link="mid_right_wheel"/>
-    <origin xyz="0 -0.2 0"/>
-    <axis xyz="0 1 0"/>
-  </joint>
-  <joint name="rr_joint" type="continuous">
-    <parent link="base_link"/>
-    <child link="rear_right_wheel"/>
-    <origin xyz="-0.25 -0.2 0"/>
-    <axis xyz="0 1 0"/>
-  </joint>
+</xacro:macro>
+  <!-- LEFT WHEELS -->
+  <xacro:wheel name="front_left_wheel" x="0.25" y="0.25"/>
+  <xacro:wheel name="mid_left_wheel" x="0" y="0.25"/>
+  <xacro:wheel name="rear_left_wheel" x="-0.25" y="0.25"/>
+  <!-- RIGHT WHEELS -->
+  <xacro:wheel name="front_right_wheel" x="0.25" y="-0.25"/>
+  <xacro:wheel name="mid_right_wheel" x="0" y="-0.25"/>
+  <xacro:wheel name="rear_right_wheel" x="-0.25" y="-0.25"/>
+  <xacro:include filename="rover.gazebo"/>
 </robot>

Commit message: Remove generated build artifacts and backup files

File: src/space_rover/urdf/rover.urdf.xacro (robot description, xacro)
@@ -1,5 +1,18 @@
 <?xml version="1.0"?>
 <robot name="rover" xmlns:xacro="http://www.ros.org/wiki/xacro">
-  <!-- BASE -->
+  <!-- ================= MATERIALS ================= -->
+  <material name="light_gray">
+    <color rgba="0.7 0.7 0.75 1"/>
+  </material>
+  <material name="accent">
+    <color rgba="0.9 0.6 0.1 1"/>
+  </material>
+  <material name="gray">
+    <color rgba="0.5 0.5 0.5 1"/>
+  </material>
+  <material name="black">
+    <color rgba="0 0 0 1"/>
+  </material>
+  <!-- ================= BASE ================= -->
   <link name="base_link">
     <visual>
@@ -7,11 +20,6 @@
         <box size="0.7 0.5 0.12"/>
       </geometry>
-	<material name="light_gray">
-  <color rgba="0.7 0.7 0.75 1"/>
-</material>
+      <material name="light_gray"/>
     </visual>
-<material name="accent">
-  <color rgba="0.9 0.6 0.1 1"/>
-</material>
     <collision>
       <geometry>
@@ -24,61 +32,42 @@
     </inertial>
   </link>
+  <!-- ================= MAST ================= -->
   <link name="mast_link">
-  <visual>
-    <geometry>
-      <cylinder radius="0.03" length="0.4"/>
-    </geometry>
-    <material name="white">
-      <color rgba="0.9 0.9 0.9 1"/>
-    </material>
-  </visual>
-</link>
-<joint name="mast_joint" type="fixed">
-  <parent link="base_link"/>
-  <child link="mast_link"/>
-  <origin xyz="0.2 0 0.3"/>
-</joint>
-  <!-- CAMERA -->
-<link name="camera_link">
-  <visual>
-    <geometry>
-      <box size="0.12 0.08 0.06"/>
-    </geometry>
-    <material name="blue">
-      <color rgba="0.1 0.3 1 1"/>
-    </material>
-  </visual>
-  <collision>
-    <geometry>
-      <box size="0.12 0.08 0.06"/>
-    </geometry>
-  </collision>
-  <inertial>
-    <mass value="0.5"/>
-    <inertia ixx="0.01" iyy="0.01" izz="0.01" ixy="0" ixz="0" iyz="0"/>
-  </inertial>
-</link>
-<link name="camera_lens">
-<visual>
-  <origin rpy="0 1.5707 0"/>
-  <geometry>
-    <cylinder radius="0.02" length="0.03"/>
-  </geometry>
-  <material name="black">
-    <color rgba="0 0 0 1"/>
-  </material>
-</visual>
-</link>
-<joint name="camera_lens_joint" type="fixed">
-  <parent link="camera_link"/>
-  <child link="camera_lens"/>
-  <origin xyz="0.06 0 0"/>
-</joint>
-<joint name="camera_joint" type="fixed">
-  <parent link="mast_link"/>
-  <child link="camera_link"/>
-  <origin xyz="0 0 0.18"/>
-</joint>
-  <!-- LIDAR -->
+    <visual>
+      <geometry>
+        <cylinder radius="0.03" length="0.4"/>
+      </geometry>
+      <material name="light_gray"/>
+    </visual>
+  </link>
+  <joint name="mast_joint" type="fixed">
+    <parent link="base_link"/>
+    <child link="mast_link"/>
+    <origin xyz="0.2 0 0.3"/>
+  </joint>
+  <!-- ================= CAMERA ================= -->
+  <link name="camera_link">
+    <visual>
+      <geometry>
+        <box size="0.12 0.08 0.06"/>
+      </geometry>
+      <material name="accent"/>
+    </visual>
+    <collision>
+      <geometry>
+        <box size="0.12 0.08 0.06"/>
+      </geometry>
+    </collision>
+    <inertial>
+      <mass value="0.5"/>
+      <inertia ixx="0.01" iyy="0.01" izz="0.01" ixy="0" ixz="0" iyz="0"/>
+    </inertial>
+  </link>
+  <joint name="camera_joint" type="fixed">
+    <parent link="mast_link"/>
+    <child link="camera_link"/>
+    <origin xyz="0 0 0.18"/>
+  </joint>
+  <!-- ================= LIDAR ================= -->
   <link name="lidar_link">
     <visual>
@@ -86,7 +75,5 @@
         <cylinder radius="0.05" length="0.05"/>
       </geometry>
-      <material name="black">
-        <color rgba="0.05 0.05 0.05 1"/>
-      </material>
+      <material name="black"/>
     </visual>
     <collision>
@@ -105,62 +92,60 @@
     <origin xyz="0 0 0.18"/>
   </joint>
+  <!-- ================= ARM ================= -->
   <link name="left_arm">
-  <visual>
-    <geometry>
-      <box size="0.4 0.05 0.05"/>
-    </geometry>
-    <material name="gray"/>
-  </visual>
-</link>
-<joint name="left_arm_joint" type="fixed">
-  <parent link="base_link"/>
-  <child link="left_arm"/>
-  <origin xyz="0 0.25 -0.05"/>
-</joint>
+    <visual>
+      <geometry>
+        <box size="0.4 0.05 0.05"/>
+      </geometry>
+      <material name="gray"/>
+    </visual>
+  </link>
+  <joint name="left_arm_joint" type="fixed">
+    <parent link="base_link"/>
+    <child link="left_arm"/>
+    <origin xyz="0 0.25 -0.05"/>
+  </joint>
+  <!-- ================= SOLAR PANEL ================= -->
   <link name="solar_panel">
-  <visual>
-    <geometry>
-      <box size="0.5 0.3 0.02"/>
-    </geometry>
-    <material name="blue_dark">
-      <color rgba="0.1 0.1 0.4 1"/>
-    </material>
-  </visual>
-</link>
-<joint name="solar_joint" type="fixed">
-  <parent link="base_link"/>
-  <child link="solar_panel"/>
-  <origin xyz="-0.1 0 0.15"/>
-</joint>
-  <!-- WHEEL MACRO -->
+    <visual>
+      <geometry>
+        <box size="0.5 0.3 0.02"/>
+      </geometry>
+      <material name="accent"/>
+    </visual>
+  </link>
+  <joint name="solar_joint" type="fixed">
+    <parent link="base_link"/>
+    <child link="solar_panel"/>
+    <origin xyz="-0.1 0 0.15"/>
+  </joint>
+  <!-- ================= WHEELS ================= -->
   <xacro:macro name="wheel" params="name x y">
-  <link name="${name}">
-    <visual>
-      <origin rpy="1.5707 0 0"/>
-      <geometry>
-        <cylinder radius="0.12" length="0.06"/>
-      </geometry>
-      <material name="wheel_black">
-        <color rgba="0.1 0.1 0.1 1"/>
-      </material>
-    </visual>
-    <collision>
-      <origin rpy="1.5707 0 0"/>
-      <geometry>
-        <cylinder radius="0.12" length="0.06"/>
-      </geometry>
-    </collision>
-    <inertial>
-      <mass value="1.0"/>
-      <inertia ixx="0.1" iyy="0.1" izz="0.1" ixy="0" ixz="0" iyz="0"/>
-    </inertial>
-  </link>
-  <joint name="${name}_joint" type="continuous">
-    <parent link="base_link"/>
-    <child link="${name}"/>
-    <origin xyz="${x} ${y} -0.12"/>
-    <axis xyz="0 1 0"/>
-  </joint>
-</xacro:macro>
+    <link name="${name}">
+      <visual>
+        <origin rpy="1.5707 0 0"/>
+        <geometry>
+          <cylinder radius="0.12" length="0.06"/>
+        </geometry>
+        <material name="black"/>
+      </visual>
+      <collision>
+        <origin rpy="1.5707 0 0"/>
+        <geometry>
+          <cylinder radius="0.12" length="0.06"/>
+        </geometry>
+      </collision>
+      <inertial>
+        <mass value="1.0"/>
+        <inertia ixx="0.1" iyy="0.1" izz="0.1" ixy="0" ixz="0" iyz="0"/>
+      </inertial>
+    </link>
+    <joint name="${name}_joint" type="continuous">
+      <parent link="base_link"/>
+      <child link="${name}"/>
+      <origin xyz="${x} ${y} -0.12"/>
+      <axis xyz="0 1 0"/>
+    </joint>
+  </xacro:macro>
   <!-- LEFT WHEELS -->
   <xacro:wheel name="front_left_wheel" x="0.25" y="0.25"/>
@@ -171,4 +156,5 @@
   <xacro:wheel name="mid_right_wheel" x="0" y="-0.25"/>
   <xacro:wheel name="rear_right_wheel" x="-0.25" y="-0.25"/>
+  <!-- INCLUDE GAZEBO FILE -->
   <xacro:include filename="rover.gazebo"/>
 </robot>

Commit message: Add navigation modules

File: src/space_rover/urdf/rover.urdf.xacro (robot description, xacro)
@@ -133,5 +133,5 @@
         <origin rpy="1.5707 0 0"/>
         <geometry>
-          <cylinder radius="0.12" length="0.06"/>
+  	<cylinder radius="0.12" length="0.06"/>
         </geometry>
       </collision>

Commit message: update nav

File: src/space_rover/urdf/rover.urdf.xacro (robot description, xacro)
@@ -90,5 +90,5 @@
     <parent link="base_link"/>
     <child link="lidar_link"/>
-    <origin xyz="0 0 0.18"/>
+    <origin xyz="0 0 0.08"/>
   </joint>
   <!-- ================= ARM ================= -->

Commit message: Improve rover sensing, obstacle avoidance, and dashboard

File: src/space_rover/urdf/rover.urdf.xacro (robot description, xacro)
@@ -36,5 +36,5 @@
     <visual>
       <geometry>
-        <cylinder radius="0.03" length="0.4"/>
+        <cylinder radius="0.022" length="0.16"/>
       </geometry>
       <material name="light_gray"/>
@@ -44,5 +44,5 @@
     <parent link="base_link"/>
     <child link="mast_link"/>
-    <origin xyz="0.2 0 0.3"/>
+    <origin xyz="0.16 0 0.14"/>
   </joint>
   <!-- ================= CAMERA ================= -->
@@ -67,5 +67,5 @@
     <parent link="mast_link"/>
     <child link="camera_link"/>
-    <origin xyz="0 0 0.18"/>
+    <origin xyz="0.18 0 0.02" rpy="0 0.14 0"/>
   </joint>
   <!-- ================= LIDAR ================= -->
@@ -90,5 +90,5 @@
     <parent link="base_link"/>
     <child link="lidar_link"/>
-    <origin xyz="0 0 0.18"/>
+    <origin xyz="0.18 0 0.035"/>
   </joint>
   <!-- ================= ARM ================= -->
